File: GPS_PND/GPS-PND/GPS-PND.kicad_pcb (KiCad board)
At the start: 2 copper layers, 56 x 20 mm, 26 parts, among them J1 ED555/2DS, U1 STM32F301K6Ux, U2 AZ1117-3.3, Y1 8Mhz

Commit message: a series of changes
Routing:
- net GND: track 6.27 -> 17.3 mm, vias 1 -> 17
- net VBAT: track 75.0 -> 75.5 mm
Changed lines of the file:
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@@
   (segment (start 157.3 94.75) (end 144.25 94.75) (width 0.25) (layer "F.Cu") (net 1))
   (segment (start 138.7 104.86) (end 138.7 98.56) (width 1) (layer "F.Cu") (net 1))
-  (segment (start 156.75 106.75) (end 156.4 106.4) (width 0.25) (layer "F.Cu") (net 1))
   (segment (start 150.75 102.25) (end 151 102.25) (width 0.25) (layer "F.Cu") (net 1))
   (segment (start 147.7625 107.6725) (end 146.0775 107.6725) (width 0.25) (layer "F.Cu") (net 1))
@@
   (segment (start 160 100) (end 160 97.45) (width 0.25) (layer "F.Cu") (net 1))
   (segment (start 144.9325 102.1825) (end 145 102.25) (width 0.25) (layer "F.Cu") (net 1))
+  (segment (start 157 106.5) (end 156.9 106.4) (width 0.25) (layer "F.Cu") (net 1))
   (segment (start 146 106) (end 146 107.75) (width 0.25) (layer "F.Cu") (net 1))
-  (segment (start 156.4 106.4) (end 156.25 106.4) (width 0.25) (layer "F.Cu") (net 1))
   (segment (start 146 102.5) (end 146.75 102.5) (width 0.25) (layer "F.Cu") (net 1))
+  (segment (start 156.9 106.4) (end 156.25 106.4) (width 0.25) (layer "F.Cu") (net 1))
   (segment (start 144.25 94.75) (end 143.25 95.75) (width 0.25) (layer "F.Cu") (net 1))
   (segment (start 160 97.45) (end 158 95.45) (width 0.25) (layer "F.Cu") (net 1))
@@
   (via (at 143.25 95.75) (size 0.6) (drill 0.3) (layers "F.Cu" "B.Cu") (free) (net 1))
   (via (at 140 101.5) (size 0.6) (drill 0.3) (layers "F.Cu" "B.Cu") (free) (net 1))
-  (via (at 156.75 106.75) (size 0.6) (drill 0.3) (layers "F.Cu" "B.Cu") (net 1))
+  (via (at 157 106.5) (size 0.6) (drill 0.3) (layers "F.Cu" "B.Cu") (net 1))
   (via (at 146.75 102.5) (size 0.6) (drill 0.3) (layers "F.Cu" "B.Cu") (net 1))
+  (segment (start 156.75 112.5) (end 157 112.25) (width 0.25) (layer "B.Cu") (net 1))
+  (segment (start 157 112.25) (end 157 106.5) (width 0.25) (layer "B.Cu") (net 1))
   (segment (start 150.5 102.5) (end 150.75 102.25) (width 0.25) (layer "B.Cu") (net 1))
   (segment (start 146.75 102.5) (end 150.5 102.5) (width 0.25) (layer "B.Cu") (net 1))
-  (segment (start 156.75 112.5) (end 156.75 106.75) (width 0.25) (layer "B.Cu") (net 1))
+  (segment (start 152.0625 102.2125) (end 152.0625 101.3125) (width 0.25) (layer "F.Cu") (net 2))
   (segment (start 136.4 103.4) (end 133 100) (width 0.25) (layer "F.Cu") (net 2))
+  (segment (start 152.0625 101.3125) (end 152 101.25) (width 0.25) (layer "F.Cu") (net 2))
+  (segment (start 152.4 105.4) (end 152.5 105.5) (width 0.25) (layer "F.Cu") (net 2))
+  (segment (start 151.375 105.4) (end 152.4 105.4) (width 0.25) (layer "F.Cu") (net 2))
+  (segment (start 156 107.525) (end 155.5625 107.0875) (width 0.25) (layer "F.Cu") (net 2))
+  (segment (start 169.5 101.25) (end 166.25 101.25) (width 0.25) (layer "F.Cu") (net 2))
   (segment (start 136.4 104.86) (end 136.4 103.4) (width 0.25) (layer "F.Cu") (net 2))
+  (segment (start 156 107.6755) (end 156 107.525) (width 0.25) (layer "F.Cu") (net 2))
+  (via (at 148.75 111.5) (size 0.6) (drill 0.3) (layers "F.Cu" "B.Cu") (net 2))
+  (via (at 162.25 97.5) (size 0.6) (drill 0.3) (layers "F.Cu" "B.Cu") (net 2))
+  (via (at 166.25 101.25) (size 0.6) (drill 0.3) (layers "F.Cu" "B.Cu") (net 2))
+  (via (at 158.25 111.25) (size 0.6) (drill 0.3) (layers "F.Cu" "B.Cu") (net 2))
   (via (at 133 100) (size 0.6) (drill 0.3) (layers "F.Cu" "B.Cu") (free) (net 2))
+  (via (at 156 109.75) (size 0.6) (drill 0.3) (layers "F.Cu" "B.Cu") (net 2))
+  (via (at 156 107.6755) (size 0.6) (drill 0.3) (layers "F.Cu" "B.Cu") (net 2))
+  (via (at 152.5 105.5) (size 0.6) (drill 0.3) (layers "F.Cu" "B.Cu") (net 2))
+  (via (at 158.5 100.25) (size 0.6) (drill 0.3) (layers "F.Cu" "B.Cu") (net 2))
+  (via (at 158.25 109.75) (size 0.6) (drill 0.3) (layers "F.Cu" "B.Cu") (net 2))
+  (via (at 155 104) (size 0.6) (drill 0.3) (layers "F.Cu" "B.Cu") (net 2))
+  (via (at 155 105.5) (size 0.6) (drill 0.3) (layers "F.Cu" "B.Cu") (net 2))
+  (via (at 152 101.25) (size 0.6) (drill 0.3) (layers "F.Cu" "B.Cu") (net 2))
+  (via (at 154 96) (size 0.6) (drill 0.3) (layers "F.Cu" "B.Cu") (net 2))
+  (via (at 147.5 105) (size 0.6) (drill 0.3) (layers "F.Cu" "B.Cu") (net 2))
+  (via (at 152.5 104) (size 0.6) (drill 0.3) (layers "F.Cu" "B.Cu") (net 2))
+  (via (at 156 111.25) (size 0.6) (drill 0.3) (layers "F.Cu" "B.Cu") (net 2))
+  (segment (start 158.5 100.25) (end 161.25 97.5) (width 0.25) (layer "B.Cu") (net 2))
+  (segment (start 161.25 97.5) (end 162.25 97.5) (width 0.25) (layer "B.Cu") (net 2))
   (segment (start 148.85 104.9) (end 151.375 104.9) (width 0.25) (layer "F.Cu") (net 3))
   (segment (start 149.5125 107.0125) (end 149.5125 107.6725) (width 0.25) (layer "F.Cu") (net 3))

Commit message: added soma changes
Parts:
- removed BOOT0, NRST: ~, Button_Switch_SMD:SW_SPST_B3U-1000P-B
- added REF**: MountingHole_2.2mm_M2_DIN965_Pad_TopBottom, MountingHole:MountingHole_2.2mm_M2_DIN965_Pad_TopBottom, F.Cu at (171.2, 94.7)
- added REF**: MountingHole_2.2mm_M2_DIN965_Pad_TopBottom, MountingHole:MountingHole_2.2mm_M2_DIN965_Pad_TopBottom, F.Cu at (171.1, 114.7)
- added SW1: ~, Button_Switch_SMD:SW_SPST_B3U-1000P-B, F.Cu at (152.2, 110.9)
- added SW2: ~, Button_Switch_SMD:SW_SPST_B3U-1000P-B, F.Cu at (152.2, 98.9)
- C6, C7, L1: moved to B.Cu
- U3: footprint GPS-PND:MS38SN3 -> Library:MS38SN4
- Y1: footprint Crystal:Crystal_SMD_0603-2Pin_6.0x3.5mm_HandSoldering -> Crystal:Crystal_SMD_3215-2Pin_3.2x1.5mm
- moved C9 10.2 mm to (148.2, 106.2), turned to 180 degrees
- moved C8 7.05 mm to (148.4, 101.1), turned to 180 degrees
- moved U3 7.01 mm to (169.0, 104.7)
- moved Y1 5.59 mm to (148.3, 103.7), turned to -90 degrees
- moved L1 4.43 mm to (149.4, 103.3)
- moved R1 2.84 mm to (155.3, 99.0), turned to -90 degrees
- moved C7 1.87 mm to (149.9, 105.6)
- moved C6 1.80 mm to (149.9, 104.6)
- moved C10 0.52 mm to (149.2, 110.9)
- moved FB2 0.15 mm to (165.5, 105.6)
- moved FB1 0.10 mm to (165.5, 104.6)
- renumbered TX to J2
Routing:
- net OSC_IN: track 15.2 -> 5.23 mm
- net GND: track 17.3 -> 8.66 mm, vias 17 -> 70
- net VBAT: track 75.5 -> 68.5 mm
- net OSC_OUT: track 11.1 -> 5.17 mm
- net NRST: track 11.8 -> 8.56 mm
- net VDDA: track 6.03 -> 3.76 mm, vias 0 -> 1
- net BOOT0: track 7.67 -> 5.47 mm
- net USART2_rX: track 16.3 -> 14.9 mm
- net USART2_tX: track 14.3 -> 13.6 mm
- net Net-(U3-RXD): track 3.70 -> 3.16 mm
Other:
- board size 56 x 20 mm -> 44.3 x 26.4 mm
- board text added: "FB1"
- board text added: "FB2"
- board text added: "TX"
- board text removed: "GNSS"
- board text removed: "GPS-PND"
